File: Hardware/Analog-Digital-Mux-Breakout.brd (EAGLE design)
At the start: 17.8 x 40.6 mm, 11 parts, among them U1 MUX-74HC4067

Commit message: Updated Revision to symbol
Parts:
- added U$2: REVISION, SparkFun-Aesthetics:REVISION
Other:
- board text added: "N. Seidle"
- board text added: "T. Klopfenstein"
- board text removed: "Revision by: T. Klopfenstein"
